File: pcb-kicad/HeadPhoneAmp/HPBooster.kicad_sch (KiCad schematic)
At the start: 6 parts, among them J1 Conn_01x03, J2 AudioJack3, J3 Conn_01x02_Socket

Commit message: Added some order infos.
Parts:
- J1: value Conn_01x03 -> ~; MFNAME (none) -> -
- J2: value AudioJack3 -> ~; MFNAME (none) -> -
- J3: value Conn_01x02_Socket -> ~; MFNAME (none) -> -
- TP1, TP2, TP3: value TestPoint -> ~; MFNAME (none) -> -
Changed lines of the file:
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@@
 			)
 		)
-		(property "Value" "AudioJack3"
+		(property "Value" "~"
 			(at 185.42 100.9649 0)
 			(effects
@@
 				)
 				(justify right)
+				(hide yes)
 			)
 		)
@@
 			)
 		)
+		(property "MFNAME" "-"
+			(at 177.8 100.33 0)
+			(effects
+				(font
+					(size 1.27 1.27)
+				)
+				(hide yes)
+			)
+		)
 		(pin "R"
 		)
@@
 			)
 		)
-		(property "Value" "TestPoint"
+		(property "Value" "~"
 			(at 168.91 95.7579 0)
 			(effects
@@
 				)
 				(justify left)
+				(hide yes)
 			)
 		)
@@
 			)
 		)
+		(property "MFNAME" "-"
+			(at 166.37 97.79 0)
+			(effects
+				(font
+					(size 1.27 1.27)
+				)
+				(hide yes)
+			)
+		)
 		(pin "1"
 		)
@@
 			)
 		)
-		(property "Value" "TestPoint"
+		(property "Value" "~"
 			(at 168.91 104.9019 0)
 			(effects
@@
 				)
 				(justify right)
+				(hide yes)
 			)
 		)
@@
 			)
 		)
+		(property "MFNAME" "-"
+			(at 166.37 100.33 0)
+			(effects
+				(font
+					(size 1.27 1.27)
+				)
+				(hide yes)
+			)
+		)
 		(pin "1"
 		)
@@
 			)
 		)
-		(property "Value" "Conn_01x02_Socket"
+		(property "Value" "~"
 			(at 79.375 72.39 0)
 			(effects
@@
 					(size 1.27 1.27)
 				)
+				(hide yes)
 			)
 		)
@@
 			)
 		)
+		(property "MFNAME" "-"
+			(at 78.74 77.47 0)
+			(effects
+				(font
+					(size 1.27 1.27)
+				)
+				(hide yes)
+			)
+		)
 		(pin "2"
 		)
@@
 			)
 		)
-		(property "Value" "Conn_01x03"
+		(property "Value" "~"
 			(at 72.39 96.52 0)
 			(effects
@@
 					(size 1.27 1.27)
 				)
+				(hide yes)
 			)
 		)
@@
 			)
 		)
+		(property "MFNAME" "-"
+			(at 72.39 102.87 0)
+			(effects
+				(font
+					(size 1.27 1.27)
+				)
+				(hide yes)
+			)
+		)
 		(pin "3"
 		)
@@
 			)
 		)
-		(property "Value" "TestPoint"
+		(property "Value" "~"
 			(at 168.91 121.4119 0)
 			(effects
@@
 				)
 				(justify right)
+				(hide yes)
 			)
 		)
@@
 			(at 166.37 116.84 0)
 			(effects
+				(font
+					(size 1.27 1.27)
+				)
+				(hide yes)
+			)
+		)
+		(property "MFNAME" "-"
+			(at 166.37 116.84 0)
+			(effects
