File: pcb-kicad/HeadPhoneAmp/PowerBoost5V12V.kicad_sch (KiCad schematic)
At the start: 39 parts, among them Q1 Q_PNP_ECB_BRT, U1 VREG_TPS6103X, U2 MCP73871

Commit message: Added some order infos.
Parts:
- B1: value BATTERY -> ~
- C1: value 10u -> 2.2u; MFNAME (none) -> EMK107BJ225KA-T
- C2, C5, C7, C8: MFNAME (none) -> EMK107BJ225KA-T
- C3, C4: MFNAME (none) -> TMK107BJ104KA-T
- C6: value C-USC1210 -> 22u; MFNAME (none) -> 293D226X96R3A2TE3
- CHRG/LBO0, DONE0, LED2: value LED0805_NOOUTLINE -> ~
- D1: MFNAME (none) -> BAT54S
- JP2: value HEADER-1X8ROUND -> ~
- L1: MFNAME (none) -> 74406042068
- LED1: value LOW-BAT -> ~
- Q1: MFNAME (none) -> MMUN2133LT1G
- R1, R3: MFNAME (none) -> RK73H1HTTCM4302D RK73H1JTTD1874F
- R13, R17, R4, R7, R9: MFNAME (none) -> RK73H1JTTD1003F
- R14, R20, R5, R8: MFNAME (none) -> RK73H1JTTD1001F
- R16: value 2k -> 1k; MFNAME (none) -> RK73H1JTTD1001F
- R2: MFNAME (none) -> RK73H1JTTD3403F
- R6: MFNAME (none) -> RK73H1JTTD2703F
- THERM0: MFNAME (none) -> RK73H1JTTD1502F
- TP1, TP3, TP5: value GND -> ~
- TP2: value 5V -> ~
- TP4: value PAD -> ~
- U1: MFNAME (none) -> TPS61090RSAR
- U2: MFNAME (none) -> MCP73871T
